File: PCB/function_generator/function_generator.kicad_sch (KiCad schematic)
At the start: 30 parts, among them J1 Barrel_Jack, J2 Buttons, J3 LCD, J4 Selector, J5 AD9833, J6 50-ohm BNC, J7 Barrel_Jack, Q1 TIP41, Q2 TIP42, SW1 SW_SPDT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

Commit message: Update
Parts:
- removed U4: LM6171, Package_DIP:DIP-8_W7.62mm, symbol Amplifier_Operational:LM7171xIN
- added U4: LM6171D, Package_SO:SOIC-8_3.9x4.9mm_P1.27mm, symbol Amplifier_Operational:LM6171D
Connections:
- net +VCC: now also U4.7 (V+)
- net -VCC: now also U4.4 (V-)
- net AD9833_VOUT: now also U4.3 (+)
- net at R7.1, RV1.2, RV1.3: now also U4.2 (-)
- net at J6.1 (In), RV1.1: now also U4.6
Changed lines of the file:
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@@
-	)
-	(symbol
-		(lib_id "Amplifier_Operational:LM7171xIN")
-		(at 219.71 120.65 0)
-		(unit 1)
-		(exclude_from_sim no)
-		(in_bom yes)
-		(on_board yes)
-		(dnp no)
-		(property "Reference" "U4"
-			(at 226.822 114.3 0)
-			(effects
-				(font
-					(size 1.27 1.27)
-				)
-			)
-		)
-		(property "Value" "LM6171"
-			(at 226.568 116.84 0)
-			(effects
-				(font
-					(size 1.27 1.27)
-				)
-			)
-		)
-		(property "Footprint" "Package_DIP:DIP-8_W7.62mm"
-			(at 219.71 120.65 0)
-			(effects
-				(font
-					(size 1.27 1.27)
-				)
-				(hide yes)
-			)
-		)
-		(property "Datasheet" "https://www.ti.com/lit/ds/symlink/lm7171.pdf"
-			(at 219.71 120.65 0)
-			(effects
-				(font
-					(size 1.27 1.27)
-				)
-				(hide yes)
-			)
-		)
-		(property "Description" "Single Very High Speed High Output Current Voltage Feedback Amplifier, DIP-8"
-			(at 219.71 120.65 0)
-			(effects
-				(font
-					(size 1.27 1.27)
-				)
-				(hide yes)
-			)
-		)
-		(pin "3"
-		)
-		(pin "7"
-		)
-		(pin "8"
-		)
-		(pin "4"
-		)
-		(pin "6"
-		)
-		(pin "2"
-		)
-		(pin "5"
-		)
-		(pin "1"
-		)
-		(instances
-			(project ""
-				(path "/bf23c2e7-f61c-45f6-a71b-5973542355b0"
-					(reference "U4")
-					(unit 1)
-				)
-			)
-		)
 	)
 	(symbol
@@
 					(unit 1)
 				)
+			)
+		)
+	)
+	(symbol
+		(lib_id "Amplifier_Operational:LM6171D")
+		(at 219.71 120.65 0)
+		(unit 1)
+		(exclude_from_sim no)
+		(in_bom yes)
+		(on_board yes)
+		(dnp no)
+		(property "Reference" "U4"
+			(at 225.044 115.57 0)
+			(effects
+				(font
+					(size 1.27 1.27)
+				)
+			)
+		)
+		(property "Value" "LM6171D"
+			(at 225.044 117.348 0)
+			(effects
+				(font
+					(size 1.27 1.27)
+				)
+			)
+		)
+		(property "Footprint" "Package_SO:SOIC-8_3.9x4.9mm_P1.27mm"
+			(at 217.17 125.73 0)
+			(effects
+				(font
+					(size 1.27 1.27)
+				)
+				(justify left)
+				(hide yes)
+			)
+		)
+		(property "Datasheet" "http://www.ti.com/lit/ds/symlink/lm6171.pdf"
+			(at 223.52 116.84 0)
+			(effects
+				(font
+					(size 1.27 1.27)
+				)
+				(hide yes)
+			)
+		)
+		(property "Description" "High Speed Low Power Low Distortion Voltage Feedback Amplifier, SOIC-8"
+			(at 219.71 120.65 0)
+			(effects
+				(font
+					(size 1.27 1.27)
+				)
+				(hide yes)
+			)
+		)
+		(pin "3"
+		)
+		(pin "2"
+		)
+		(pin "7"
+		)
+		(pin "6"
+		)
+		(pin "1"
+		)
+		(pin "5"
+		)
+		(pin "8"
+		)
+		(pin "4"
+		)
+		(instances
+			(project ""
+				(path "/bf23c2e7-f61c-45f6-a71b-5973542355b0"
+					(reference "U4")
+					(unit 1)
+				)

Commit message: Update
Parts:
- U4: value LM6171D -> LM6171
