File: PCB/function_generator/function_generator.kicad_pcb (KiCad board)
At the start: 2 copper layers, 65 x 85 mm, 30 parts, among them J1 Barrel_Jack, J2 Buttons, J3 LCD, J4 Selector, J5 AD9833, J6 50-ohm BNC, J7 Barrel_Jack, Q1 TIP41, Q2 TIP42, SW1 SW_SPDT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

Commit message: Update
Parts:
- U4: value LM6171 -> LM6171D; footprint Package_DIP:DIP-8_W7.62mm -> Package_SO:SOIC-8_3.9x4.9mm_P1.27mm
- moved U4 5.03 mm to (123.7, 79.8)
Routing:
- net +VCC: track 164.9 -> 171.2 mm, vias 1 -> 2
- net /AD9833_VOUT: track 64.4 -> 69.0 mm, vias 3 -> 4
- net +3.3V: track 119.1 -> 122.8 mm
- net Net-(J6-In): track 92.0 -> 94.8 mm
- net Net-(U4--): track 83.2 -> 84.7 mm, vias 0 -> 1
- net -VCC: track 210.3 -> 209.5 mm, vias 4 -> 6
Other:
- board text added: "RJX Function Generator"

Commit message: Update
Routing:
- net +VCC: track 171.2 -> 167.3 mm
- net -VCC: track 209.5 -> 205.9 mm
- net +3.3V: track 122.8 -> 119.9 mm
- net GND: track 310.8 -> 308.5 mm
- net Net-(J7-Pad1): track 104.4 -> 105.8 mm

Commit message: Update
Parts:
- U4: value LM6171D -> LM6171

Commit message: Update
Routing:
- net -VCC: track 205.9 -> 207.1 mm
Changed lines of the file:
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@@
 		)
 		(property "Value" "LM6171"
-			(at 0 3.4 90)
+			(at 0.055 3.335 90)
 			(layer "F.SilkS")
 			(effects
@@
 	)
 	(segment
+		(start 125.62 81.22)
+		(end 125.61 81.23)
+		(width 0.5)
+		(layer "F.Cu")
+		(net 3)
+	)
+	(segment
 		(start 127.98 95.47)
 		(end 128.45 95)
@@
 	)
 	(segment
-		(start 127.543599 81.215)
-		(end 125.625 81.215)
-		(width 0.5)
-		(layer "F.Cu")
-		(net 3)
-	)
-	(segment
 		(start 141.41 105.04)
 		(end 141.6 105.23)
@@
 	)
 	(segment
-		(start 125.625 81.215)
-		(end 125.61 81.23)
-		(width 0.5)
-		(layer "F.Cu")
-		(net 3)
-	)
-	(segment
 		(start 131.64 121.24)
 		(end 131.64 129.03)
@@
 	)
 	(segment
+		(start 128.49 81.22)
+		(end 128.51 81.24)
+		(width 0.25)
+		(layer "F.Cu")
+		(net 3)
+	)
+	(segment
 		(start 127.98 96.03)
 		(end 127.98 95.47)
@@
 	)
 	(segment
-		(start 127.98 96.03)
-		(end 127.98 113.77)
+		(start 128.01 81.22)
+		(end 125.62 81.22)
 		(width 0.5)
 		(layer "F.Cu")
@@
 	)
 	(segment
-		(start 125.61 81.23)
-		(end 125.61 82.3)
+		(start 127.98 96.03)
+		(end 127.98 113.77)
 		(width 0.5)
 		(layer "F.Cu")
@@
 	)
 	(segment
+		(start 125.61 81.23)
+		(end 125.61 82.3)
+		(width 0.5)
+		(layer "F.Cu")
+		(net 3)
+	)
+	(segment
 		(start 112.29 67.94)
 		(end 113.85 69.5)
@@
 	)
 	(segment
+		(start 128.01 81.22)
+		(end 128.49 81.22)
+		(width 0.5)
+		(layer "F.Cu")
+		(net 3)
+	)
+	(segment
 		(start 144.8 97.05)
 		(end 144.75 97)
@@
 	)
 	(via
-		(at 144.75 97)
+		(at 128.51 81.24)
 		(size 0.6)
 		(drill 0.3)
@@
 	)
 	(via
-		(at 133.647702 87.747702)
+		(at 144.75 97)
 		(size 0.6)
 		(drill 0.3)
@@
 	)
 	(via
-		(at 127.543599 81.215)
+		(at 133.647702 87.747702)
 		(size 0.6)
 		(drill 0.3)
@@
 	)
 	(segment
+		(start 128.51 81.24)
+		(end 128.9 80.85)
+		(width 0.5)
+		(layer "B.Cu")
+		(net 3)
+	)
+	(segment
+		(start 128.9 80.85)
+		(end 128.9 71.99)
+		(width 0.5)
+		(layer "B.Cu")
+		(net 3)
+	)
+	(segment
 		(start 121.4 118.387677)
 		(end 121.4 135.1)
@@
 	)
 	(segment
-		(start 127.543599 81.215)
-		(end 127.705 81.215)
-		(width 0.5)
-		(layer "B.Cu")
-		(net 3)
-	)
-	(segment
 		(start 123.74 116.047677)
 		(end 121.4 118.387677)
@@
 	)
 	(segment
+		(start 128.44 71.53)
+		(end 128.17 71.53)
+		(width 0.5)
+		(layer "B.Cu")
+		(net 3)
+	)
+	(segment
 		(start 111.51 118.39)
 		(end 113.29 118.39)
@@
 	)
 	(segment
-		(start 127.705 81.215)
-		(end 128.17 80.75)
-		(width 0.5)
-		(layer "B.Cu")
-		(net 3)
-	)
-	(segment
 		(start 110.2 134.9)
 		(end 110.2 119.7)
@@
 	)
 	(segment
-		(start 128.17 80.75)
-		(end 128.17 71.53)
+		(start 128.9 71.99)
+		(end 128.44 71.53)
 		(width 0.5)
 		(layer "B.Cu")
@@
 	)
 	(segment
+		(start 146.83 108.45)
+		(end 146.86 108.48)
+		(width 0.5)
+		(layer "F.Cu")
+		(net 5)
+	)
+	(segment
 		(start 163.62 76.28)
 		(end 164.21 75.69)
@@
 	)
 	(segment
+		(start 146.83 105.49)
+		(end 146.83 108.45)
+		(width 0.5)
+		(layer "F.Cu")
+		(net 5)
+	)
+	(segment
 		(start 138.2 123.8)
 		(end 139.15 123.8)
@@
 	)
 	(segment
+		(start 150.6 98.78)
+		(end 150.6 101.72)
+		(width 0.5)
+		(layer "F.Cu")
+		(net 5)
+	)
+	(segment
 		(start 150.64 111.83)
 		(end 150.64 110.71)
@@
 	)
 	(segment
+		(start 150.6 101.72)
+		(end 146.83 105.49)
+		(width 0.5)
+		(layer "F.Cu")
+		(net 5)
+	)
+	(segment
 		(start 141.3 124.05)
 		(end 141.3 126.45)
@@
 	)
 	(segment
-		(start 150.6 100.75)
-		(end 148.65 102.7)
-		(width 0.5)
-		(layer "F.Cu")
-		(net 5)
-	)
-	(segment
 		(start 165.84 63.59)
 		(end 165.84 66.13)
@@
 	)
 	(segment
-		(start 150.6 98.78)
-		(end 150.6 100.75)
-		(width 0.5)
-		(layer "F.Cu")
-		(net 5)
-	)
-	(segment
 		(start 125.29 122.597677)
 		(end 123.74 121.047677)
@@
 	)
 	(segment
-		(start 146.9 104.45)
-		(end 146.9 106.4)
-		(width 0.5)
-		(layer "F.Cu")
-		(net 5)
-	)
-	(segment
 		(start 157.555 109.915)
 		(end 157.93 110.29)
@@
 	)
 	(segment
-		(start 148.65 102.7)
-		(end 146.9 104.45)
-		(width 0.5)
-		(layer "F.Cu")
-		(net 5)
-	)
-	(segment
 		(start 116.88 131.49)
 		(end 119.39 128.98)
@@
 	)
 	(via
-		(at 146.9 106.4)
+		(at 146.86 108.48)
 		(size 0.6)
 		(drill 0.3)
@@
 	)
 	(segment
+		(start 146.86 108.48)
+		(end 146.9 108.52)
+		(width 0.5)
+		(layer "B.Cu")
+		(net 5)
+	)
+	(segment
 		(start 111.25 115.85)
 		(end 109.85 114.45)
@@
 	)
 	(segment
-		(start 126.9 91)
-		(end 127.98 89.92)
+		(start 147.15 118.23)
+		(end 147.38 118.23)
 		(width 0.5)
 		(layer "B.Cu")
@@
 	)
 	(segment
-		(start 146.9 106.4)
-		(end 146.9 117.98)
+		(start 126.9 91)
+		(end 127.98 89.92)
 		(width 0.5)
 		(layer "B.Cu")
@@
 	)
 	(segment
-		(start 127.98 89.92)
-		(end 127.98 88.41)
+		(start 146.9 108.52)
+		(end 146.9 117.98)
 		(width 0.5)
 		(layer "B.Cu")
@@
 	)
 	(segment
-		(start 122.9 92.15)
-		(end 124.05 91)
+		(start 127.98 89.92)
+		(end 127.98 88.41)
 		(width 0.5)
 		(layer "B.Cu")
@@
 	)
 	(segment
-		(start 147.15 118.23)
-		(end 147.38 118.23)
+		(start 122.9 92.15)
+		(end 124.05 91)
 		(width 0.5)
 		(layer "B.Cu")
@@
 	)
 	(segment
+		(start 146.9 117.98)
+		(end 147.15 118.23)
+		(width 0.5)
+		(layer "B.Cu")
+		(net 5)
+	)
+	(segment
 		(start 109.85 104.55)
 		(end 110.9 103.5)
@@
 		(width 0.5)
 		(layer "B.Cu")
-		(net 5)
-	)
-	(segment
-		(start 146.9 117.98)
-		(end 147.15 118.23)
-		(width 0.5)
-		(layer "B.Cu")
